File: rpmled3.sch (KiCad schematic (older format))
At the start: 41 parts, among them J1 Conn_01x02, J2 Conn_01x04, J3 Conn_01x02, J4 Conn_01x02, J7 Conn_01x02, U1 STP16C596, U2 STM32F042K6Tx, U3 STP16C596, U4 SN65HVD230, U5 ST1S14PHR_MY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

Commit message: Не стандартные компоненты перенесены в локальную библиотеку Исправления v0.1.2
Parts:
- D1, D2, D3, D4, D5, D6, D7, D8: footprint posad:RGB_LEB_InLine -> rpmledlib:RGB_LEB_InLine
Changed lines of the file:
@@
 F 0 "D1" V 1600 1600 50  0000 R CNN
 F 1 "LED_ARGB" V 1600 1250 50  0000 R CNN
-F 2 "posad:RGB_LEB_InLine" H 1400 1300 50  0001 C CNN
+F 2 "rpmledlib:RGB_LEB_InLine" H 1400 1300 50  0001 C CNN
 F 3 "~" H 1400 1300 50  0001 C CNN
 	1    1400 1350
@@
 F 0 "D2" V 2400 1550 50  0000 R CNN
 F 1 "LED_ARGB" V 2400 1200 50  0000 R CNN
-F 2 "posad:RGB_LEB_InLine" H 2200 1300 50  0001 C CNN
+F 2 "rpmledlib:RGB_LEB_InLine" H 2200 1300 50  0001 C CNN
 F 3 "~" H 2200 1300 50  0001 C CNN
 	1    2200 1350
@@
 F 0 "D3" V 3200 1500 50  0000 R CNN
 F 1 "LED_ARGB" V 3200 1250 50  0000 R CNN
-F 2 "posad:RGB_LEB_InLine" H 3000 1300 50  0001 C CNN
+F 2 "rpmledlib:RGB_LEB_InLine" H 3000 1300 50  0001 C CNN
 F 3 "~" H 3000 1300 50  0001 C CNN
 	1    3000 1350
@@
 F 0 "D4" V 4050 1550 50  0000 R CNN
 F 1 "LED_ARGB" V 4050 1250 50  0000 R CNN
-F 2 "posad:RGB_LEB_InLine" H 3850 1300 50  0001 C CNN
+F 2 "rpmledlib:RGB_LEB_InLine" H 3850 1300 50  0001 C CNN
 F 3 "~" H 3850 1300 50  0001 C CNN
 	1    3850 1350
@@
 F 0 "D5" V 4900 1550 50  0000 R CNN
 F 1 "LED_ARGB" V 4900 1250 50  0000 R CNN
-F 2 "posad:RGB_LEB_InLine" H 4700 1300 50  0001 C CNN
+F 2 "rpmledlib:RGB_LEB_InLine" H 4700 1300 50  0001 C CNN
 F 3 "~" H 4700 1300 50  0001 C CNN
 	1    4700 1350
@@
 F 0 "D6" V 5750 1550 50  0000 R CNN
 F 1 "LED_ARGB" V 5750 1200 50  0000 R CNN
-F 2 "posad:RGB_LEB_InLine" H 5550 1300 50  0001 C CNN
+F 2 "rpmledlib:RGB_LEB_InLine" H 5550 1300 50  0001 C CNN
 F 3 "~" H 5550 1300 50  0001 C CNN
 	1    5550 1350
@@
 F 0 "D7" V 6650 1500 50  0000 R CNN
 F 1 "LED_ARGB" V 6650 1200 50  0000 R CNN
-F 2 "posad:RGB_LEB_InLine" H 6450 1300 50  0001 C CNN
+F 2 "rpmledlib:RGB_LEB_InLine" H 6450 1300 50  0001 C CNN
 F 3 "~" H 6450 1300 50  0001 C CNN
 	1    6450 1350
@@
 F 0 "D8" V 7500 1500 50  0000 R CNN
 F 1 "LED_ARGB" V 7500 1250 50  0000 R CNN
-F 2 "posad:RGB_LEB_InLine" H 7300 1300 50  0001 C CNN
+F 2 "rpmledlib:RGB_LEB_InLine" H 7300 1300 50  0001 C CNN
 F 3 "~" H 7300 1300 50  0001 C CNN
 	1    7300 1350
